File: quadcopter.sch (EAGLE design)
At the start: 40 parts, among them J1 ISP, J3 POWER_JACKPTH_LOCK, U1 ATMEGA128RFA1, U2 LM1117, Y1 16MHz

Commit message: almost forgot to include schematic
Parts:
- removed C10, C14: 10uF, SparkFun-Passives:CAP_POL1206
- removed C12: 1uF, SparkFun-Passives:CAP0402-CAP
- removed C13: 0.1uF, SparkFun-Passives:CAP0402-CAP
- removed FID1, FID2: FIDUCIALUFIDUCIAL, SparkFun-Aesthetics:FIDUCIALUFIDUCIAL
- removed J3: POWER_JACKPTH_LOCK, SparkFun-Connectors:POWER_JACKPTH_LOCK
- removed JP10, JP4: LOGO-SFENEW, SparkFun-Aesthetics:LOGO-SFENEW
- removed JP6: (no value), SparkFun-Connectors:M02JST-PTH-2
- removed JP7: (no value), SparkFun-Connectors:M021X02_NO_SILK
- removed JP8: (no value), SparkFun-Connectors:M023.5MM-NO_SILK
- removed LED1: RED, SparkFun-LED:LED0603
- removed LED2, LED3: GREEN, SparkFun-LED:LED0603
- removed R2: 1k, SparkFun-Passives:RESISTOR0402-RES
- removed R3: 240, SparkFun:RESISTOR0402-RES
- removed R4: 390, SparkFun:RESISTOR0402-RES
- removed R5, R6: 330, quadparts_prebuilt:RESISTOR_SMD-2012-0805-330
- removed S2: (no value), SparkFun:SWITCH-SPST-SMD-A
- removed U2: LM1117, SparkFun:V_REG_317SMD
- added BATT1: BATTERY-HUBSAN-W/HOLDER, quadparts_prebuilt:BATTERY-HUBSAN-W/HOLDER
- added C11, C15, C16: 0.1uF, quadparts_prebuilt:CAPACITOR-NP_SMD-2012-0805_CERAMIC-0.1UF
- added C17: 10uF, quadparts_prebuilt:CAPACITOR-NP_SMD-2012-0805_CERAMIC-10UF
- added C18: 0.01uF, quadparts_prebuilt:CAPACITOR-NP_SMD-2012-0805_CERAMIC-0.01UF
- added C19, C20, C21, C22, C23, C24, C25, C26: 100uf, capacitor-wima:C10/4
- added C27, C28: 1uF, quadparts_prebuilt:CAPACITOR-NP_SMD-2012-0805_CERAMIC-1UF
- added D1, D2: green, quadparts_prebuilt:DIODE-LED_SMD-2012-0805-GREEN
- added D3, D4, D5, D6: 20V-500MA, quadparts_prebuilt:DIODE-SCHOTTKY_SMD-SOD123-360MV
- added J2: (no value), quadparts_prebuilt:SIP-10_TH-254X10-1
- added J4: (no value), quadparts_michael:MALE_HEADER_2POS-2X1-0.1IN
- added Q1, Q2, Q3, Q4: (no value), Lab2:MOSFET-SI2302CDS-T1-E3
- added R10, R11, R12, R13, R14, R15, R16, R9: 100R, Lab5:R-US_R0805
- added R7, R8: 5.1K, quadparts_prebuilt:RESISTOR_SMD-2012-0805-5.1K
- added STEP_DOWN: TPS73633-DBVT, quadparts_prebuilt:TPS73633-DBVT
- added U$2: LSM9DS1TR_IMU-9_AXIS, quadparts_michael:LSM9DS1TR_IMU-9_AXIS
- added U$3, U$4, U$5: MOTOR_PADS, quadparts_prebuilt:MOTOR_PADS
- added U$6: NET_BRIDGE, quadparts_michael:NET_BRIDGE
- U$1: value OSHW-LOGOS -> MOTOR_PADS; device SparkFun-Aesthetics:OSHW-LOGOS -> quadparts_prebuilt:MOTOR_PADS
Connections:
- removed net 3.3V: C10.+, C12.1, C3.1, C4.1, R1.2, R2.2, R3.2, U1.DEVDD, U1.EVDD, U2.OUT
- removed net FB: R3.1, R4.2, U2.ADJ
- removed net N$13: LED2.A, R6.1
- removed net N$2: LED1.A, R2.1
- removed net N$8: LED3.A, R5.1
- removed net N$9: J3.PWR, JP6.2, JP7.2, JP8.2, S2.P
- new net 3V: C11.1, C16.1, C17.1, C28.1, J2.7, R7.1, R8.1, STEP_DOWN.OUT, U$2.P$1.VDDIO, U$2.P$22.VDD, U$2.P$23.VDD, U$2.P$3.VDDIO
- new net BAT_GND: BATT1.N
- new net FILTERED: Q2.G, R10.1, R9.2
- new net FILTERED1: Q1.G, R11.2, R12.1
- new net FILTERED3: Q4.G, R15.2, R16.1
- new net FILTERED5: Q3.G, R13.2, R14.1
- new net FLYBACK: D3.A, Q2.D, U$1.V-
- new net FLYBACK1: D4.A, Q1.D, U$3.V-
- new net FLYBACK3: D6.A, Q4.D, U$5.V-
- new net FLYBACK5: D5.A, Q3.D, U$4.V-
- new net N$1: BATT1.P, J4.2
- new net N$10: C20.2, Q2.S
- new net N$14: C22.2, Q1.S
- new net N$15: C24.2, Q3.S
- new net N$16: C26.2, Q4.S
- new net N$17: U$2.P$6.SDO_M, U$2.P$7.CS_A/G, U$2.P$8.CS_M
- new net N$21: C27.1, STEP_DOWN.IN
- new net N$22: STEP_DOWN.GND
- new net N$23: U1.DEVDD, U1.EVDD
- new net N$24: R1.2
- new net N$25: C4.1
- new net N$26: C3.1
- new net N$27: STEP_DOWN.EN
- new net N$5: C18.2, U$2.P$21.CAP
- new net N$6: C15.2, U$2.P$24.C1
- new net PWM-PB5: C20.1, R9.1
- new net PWM-PE3: C26.1, R15.1
- new net PWM-PE4: C22.1, R11.1
- new net PWM-PE5: C24.1, R13.1
- net GND: now also C11.2, C15.1, C16.2, C17.2, C18.1, C19.2, C21.2, C23.2, C25.2, C27.2, C28.2, D1.C, D2.C, J2.10, J2.9, R10.2, R12.2, R14.2, R16.2, U$2.P$14.RES, U$2.P$15.RES, U$2.P$16.RES, U$2.P$17.RES, U$2.P$18.RES, U$2.P$19.GND, U$2.P$20.GND; no longer C10.-, C12.2, C13.2, C14.-, J3.GND, J3.GNDBREAK, JP6.1, JP7.1, JP8.1, LED1.C, LED2.C, LED3.C, R4.1
- net PB6: no longer R5.2
- net PB7: no longer R6.2
- net SCL: now also R7.2, U$2.P$2.SLC/SCP
- net SDA: now also R8.2, U$2.P$4.SDA/SDI/SDO
- net VCC: now also C19.1, C21.1, C23.1, C25.1, D1.A, D2.A, D3.C, D4.C, D5.C, D6.C, J2.8, J4.1, U$1.V+, U$3.V+, U$4.V+, U$5.V+; no longer C13.1, C14.+, S2.O, U2.IN
Other:
- note added: "Filter"
- note added: "Flyback"
- note removed: "800mA"
- note removed: "ADJ - 3V -- TODO: Redesign"
- note removed: "I think I'm supposed to replace this with our microcontroller"
- note removed: "Jim Lindblom"
- note removed: "v23"
- moved on the sheet: A1, B1, C1, C2, C3, C4, C5, C6, C7, C8, C9, J1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

Commit message: fixed stuff from design review
Parts:
- removed A1: ANTENNA2SMD5, SparkFun-RF:ANTENNA2SMD5
- removed B1: 748421245, SparkFun-RF:BALUN0805
- removed C19, C20, C21, C22, C26: 100uf, capacitor-wima:C10/4
- removed C9: 0.1uF, quadparts_prebuilt:CAPACITOR-NP_SMD-2012-0805_CERAMIC-0.1UF
- removed D2: green, quadparts_prebuilt:DIODE-LED_SMD-2012-0805-GREEN
- removed D4: 20V-500MA, quadparts_prebuilt:DIODE-SCHOTTKY_SMD-SOD123-360MV
- removed JP1, JP9: FTDI, SparkFun-Connectors:FTDI_BASICPTH
- removed Q1, Q2, Q3, Q4: (no value), Lab2:MOSFET-SI2302CDS-T1-E3
- removed R11, R12, R13, R14, R9: 100R, Lab5:R-US_R0805
- removed U$4: MOTOR_PADS, quadparts_prebuilt:MOTOR_PADS
- removed U$6: NET_BRIDGE, quadparts_michael:NET_BRIDGE
- removed Y1: 16MHz, SparkFun-FreqCtrl:CRYSTAL5X3
- added B2: BALUN0805, quadparts_prebuilt:BALUN0805
- added C10, C12, C30, C34: 0.1uF, quadparts_prebuilt:CAPACITOR-NP_SMD-2012-0805_CERAMIC-0.1UF
- added C13: 0.01uF, quadparts_prebuilt:CAPACITOR-NP_SMD-2012-0805_CERAMIC-0.01UF
- added C29, C33: 100uf, capacitor-wima:C10/4
- added D11, D9: 20V-500MA, quadparts_prebuilt:DIODE-SCHOTTKY_SMD-SOD123-360MV
- added JP3, JP4: FTDI_BASICPTH, quadparts_prebuilt:FTDI_BASICPTH
- added R17, R2, R21, R23: 10K, quadparts_prebuilt:RESISTOR_SMD-2012-0805-10K
- added R20, R22: 100R, Lab5:R-US_R0805
- added R3: 330, quadparts_prebuilt:RESISTOR_SMD-2012-0805-330
- added U$13, U$17, U$19: MOTOR_PADS, quadparts_prebuilt:MOTOR_PADS
- added U$16, U$18, U$20, U$7: MOSFET-N_CHANNEL, quadparts_michael:MOSFET-N_CHANNEL
- added Y2: (no value), quadparts_prebuilt:CRYSTAL5X3
- C24: value 100uf -> 0.1uF; device capacitor-wima:C10/4 -> quadparts_prebuilt:CAPACITOR-NP_SMD-2012-0805_CERAMIC-0.1UF
- D1: value green -> (none); device quadparts_prebuilt:DIODE-LED_SMD-2012-0805-GREEN -> quadparts_michael:LED-RED
- D3: value 20V-500MA -> (none); device quadparts_prebuilt:DIODE-SCHOTTKY_SMD-SOD123-360MV -> quadparts_michael:LED-RED
- R10: value 100R -> 10K; device Lab5:R-US_R0805 -> quadparts_prebuilt:RESISTOR_SMD-2012-0805-10K
- R7: value 5.1K -> 10K; device quadparts_prebuilt:RESISTOR_SMD-2012-0805-5.1K -> quadparts_prebuilt:RESISTOR_SMD-2012-0805-10K
- R8: value 5.1K -> 330; device quadparts_prebuilt:RESISTOR_SMD-2012-0805-5.1K -> quadparts_prebuilt:RESISTOR_SMD-2012-0805-330
- U$1: value MOTOR_PADS -> LSM9DS1TR_IMU-9_AXIS; device quadparts_prebuilt:MOTOR_PADS -> quadparts_michael:LSM9DS1TR_IMU-9_AXIS
- U$2: value LSM9DS1TR_IMU-9_AXIS -> NET_BRIDGE; device quadparts_michael:LSM9DS1TR_IMU-9_AXIS -> quadparts_michael:NET_BRIDGE
- U$3: value MOTOR_PADS -> ANTENNA2SMD5; device quadparts_prebuilt:MOTOR_PADS -> quadparts_prebuilt:ANTENNA2SMD5
Connections:
- removed net DTR: C9.1, JP9.1
- removed net N$14: C22.2, Q1.S
- removed net PWM-PB5: C20.1, R9.1
- removed net PWM-PE3: C26.1, R15.1
- removed net PWM-PE4: C22.1, R11.1
- removed net PWM-PE5: C24.1, R13.1
- removed net VCC: C19.1, C21.1, C23.1, C25.1, D1.A, D2.A, D3.C, D4.C, D5.C, D6.C, J2.8, J4.1, U$1.V+, U$3.V+, U$4.V+, U$5.V+
- new net N$12: D1.C, R3.2
- new net N$18: C30.2, U$18.S
- new net N$2: C13.1, STEP_DOWN.NC/FB
- new net N$28: C34.2, U$20.S
- new net N$8: JP3.6, JP4.6
- new net N$9: C12.1, JP3.1
- new net VBAT: C23.1, C25.1, C29.1, C33.1, D1.A, D11.C, D3.A, D5.C, D6.C, D9.C, J2.8, J4.1, U$13.V+, U$17.V+, U$19.V+, U$5.V+
- net 3V: now also R2.1, U$1.P$1.VDDIO, U$1.P$13.DEN_A/G, U$1.P$22.VDD, U$1.P$23.VDD, U$1.P$3.VDDIO, U$1.P$5.SDO_A/G; no longer R8.1, U$2.P$1.VDDIO, U$2.P$22.VDD, U$2.P$23.VDD, U$2.P$3.VDDIO
- net BAT_GND: now also C27.2, J2.10, U$2.P$2
- net FILTERED: now also C24.1, R16.2, R17.2, U$16.G; no longer Q2.G, R10.1, R9.2
- net FILTERED1: now also C30.1, R20.2, R21.2, U$18.G; no longer Q1.G, R11.2, R12.1
- net FILTERED3: now also C10.1, R10.2, U$7.G; no longer Q4.G, R16.1
- net FILTERED5: now also C34.1, R22.2, R23.2, U$20.G; no longer Q3.G, R13.2, R14.1
- net FLYBACK: now also D5.A, U$13.V-, U$16.D; no longer D3.A, Q2.D, U$1.V-
- net FLYBACK1: now also D9.A, U$17.V-, U$18.D; no longer D4.A, Q1.D, U$3.V-
- net FLYBACK3: now also U$7.D; no longer Q4.D
- net FLYBACK5: now also D11.A, U$19.V-, U$20.D; no longer D5.A, Q3.D, U$4.V-
- net GND: now also B2.GND@5, C13.2, C29.2, C33.2, R10.1, R17.1, R21.1, R23.1, R3.1, R8.1, U$1.P$14.RES, U$1.P$15.RES, U$1.P$16.RES, U$1.P$17.RES, U$1.P$18.RES, U$1.P$19.GND, U$1.P$20.GND, U$2.P$1; no longer B1.GND@5, C19.2, C21.2, C27.2, D1.C, D2.C, J2.10, JP1.6, JP9.6, R10.2, R12.2, R14.2, R16.2, U$2.P$14.RES, U$2.P$15.RES, U$2.P$16.RES, U$2.P$17.RES, U$2.P$18.RES, U$2.P$19.GND, U$2.P$20.GND
- net N$10: now also D3.C, R8.2; no longer C20.2, Q2.S
- net N$15: now also U$16.S; no longer Q3.S
- net N$16: now also C10.2, U$7.S; no longer C26.2, Q4.S
- net N$17: now also U$1.P$6.SDO_M, U$1.P$7.CS_A/G, U$1.P$8.CS_M; no longer U$2.P$6.SDO_M, U$2.P$7.CS_A/G, U$2.P$8.CS_M
- net N$3: now also Y2.2; no longer Y1.2
- net N$4: now also Y2.1; no longer Y1.1
- net N$5: now also U$1.P$21.CAP; no longer U$2.P$21.CAP
- net N$6: now also U$1.P$24.C1; no longer U$2.P$24.C1
- net N$7: now also B2.GND@2; no longer B1.GND@2
- net PB5: now also R16.1
- net PE3: now also R15.1
- net PE4: now also R20.1
- net PE5: now also R22.1
- net RESET: now also C12.2; no longer C9.2
- net RFANT: now also B2.IN, U$3.SIGNAL; no longer A1.SIGNAL, B1.IN
- net RFN: now also B2.OUT2; no longer B1.OUT2
- net RFP: now also B2.OUT1; no longer B1.OUT1
- net RXD1: now also JP3.2, JP4.2; no longer JP1.3, JP9.3
- net SCL: now also R2.2, U$1.P$2.SCL/SCP; no longer R7.2, U$2.P$2.SLC/SCP
- net SDA: now also R7.2, U$1.P$4.SDA/SDI/SDO; no longer R8.2, U$2.P$4.SDA/SDI/SDO
- net TXD1: now also JP3.3, JP4.3; no longer JP1.2, JP9.2
Other:
- note added: "Design review said SDO_M should be set low, but talked with person with advice from prof, and prof said set high. This sets less significant bit, not necessarily the least sig bit"
- note added: "SDO_A/G should be set high to enable I2C"
- note removed: "Flyback"
- moved on the sheet: C23, C25, D5, R10, R15, R16, R7, R8, U$5

Commit message: trying to work with pour, but can't move to internal layer. don't know why :(
Connections:
- removed net N$15: C24.2, U$16.S
- removed net N$16: C10.2, U$7.S
- removed net N$18: C30.2, U$18.S
- removed net N$28: C34.2, U$20.S
- net GND: now also C10.2, C24.2, C30.2, C34.2, U$16.S, U$18.S, U$20.S, U$7.S
Other:
- moved on the sheet: R21
Changed lines of the file:
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@@
 <?xml version="1.0" encoding="utf-8"?>
 <!DOCTYPE eagle SYSTEM "eagle.dtd">
-<eagle version="8.1.0">
+<eagle version="8.1.1">
 <drawing>
 <settings>
@@
 <layers>
 <layer number="1" name="Top" color="4" fill="1" visible="no" active="no"/>
+<layer number="2" name="Route2" color="1" fill="3" visible="no" active="no"/>
+<layer number="3" name="Route3" color="4" fill="3" visible="no" active="no"/>
+<layer number="4" name="Route4" color="1" fill="4" visible="no" active="no"/>
+<layer number="5" name="Route5" color="4" fill="4" visible="no" active="no"/>
+<layer number="6" name="Route6" color="1" fill="8" visible="no" active="no"/>
+<layer number="7" name="Route7" color="4" fill="8" visible="no" active="no"/>
+<layer number="8" name="Route8" color="1" fill="2" visible="no" active="no"/>
+<layer number="9" name="Route9" color="4" fill="2" visible="no" active="no"/>
+<layer number="10" name="Route10" color="1" fill="7" visible="no" active="no"/>
+<layer number="11" name="Route11" color="4" fill="7" visible="no" active="no"/>
+<layer number="13" name="Route13" color="4" fill="5" visible="no" active="no"/>
+<layer number="14" name="Route14" color="1" fill="6" visible="no" active="no"/>
+<layer number="15" name="Route15" color="4" fill="6" visible="no" active="no"/>
 <layer number="16" name="Bottom" color="1" fill="1" visible="no" active="no"/>
 <layer number="17" name="Pads" color="2" fill="1" visible="no" active="no"/>
@@
 <instance part="J2" gate="G$1" x="-38.1" y="134.62"/>
 <instance part="STEP_DOWN" gate="G$1" x="33.02" y="142.24"/>
-<instance part="GND38" gate="1" x="226.06" y="-12.7"/>
+<instance part="GND38" gate="1" x="223.52" y="-15.24"/>
 <instance part="GND39" gate="1" x="226.06" y="20.32"/>
 <instance part="C25" gate="G$1" x="226.06" y="30.48"/>
@@
 <instance part="R8" gate="G$1" x="-48.26" y="-30.48" rot="R90"/>
 <instance part="R10" gate="G$1" x="241.3" y="-5.08" rot="R90"/>
-<instance part="GND35" gate="1" x="236.22" y="101.6"/>
+<instance part="GND35" gate="1" x="233.68" y="99.06"/>
 <instance part="GND36" gate="1" x="236.22" y="134.62"/>
 <instance part="C23" gate="G$1" x="236.22" y="144.78"/>
@@
 <instance part="U$16" gate="G$1" x="266.7" y="109.22" rot="R90"/>
 <instance part="R17" gate="G$1" x="251.46" y="109.22" rot="R90"/>
-<instance part="GND37" gate="1" x="-99.06" y="99.06"/>
+<instance part="GND37" gate="1" x="-101.6" y="96.52"/>
 <instance part="GND40" gate="1" x="-99.06" y="132.08"/>
 <instance part="C29" gate="G$1" x="-99.06" y="142.24"/>
@@
 <instance part="C30" gate="G$1" x="-93.98" y="109.22"/>
 <instance part="U$18" gate="G$1" x="-68.58" y="106.68" rot="R90"/>
-<instance part="R21" gate="G$1" x="-83.82" y="106.68" rot="R90"/>
-<instance part="GND46" gate="1" x="-101.6" y="-45.72"/>
+<instance part="R21" gate="G$1" x="-83.82" y="104.14" rot="R90"/>
+<instance part="GND46" gate="1" x="-104.14" y="-48.26"/>
 <instance part="GND47" gate="1" x="-101.6" y="-12.7"/>
 <instance part="C33" gate="G$1" x="-101.6" y="-2.54"/>
@@
 <segment>
 <pinref part="GND4" gate="1" pin="GND"/>
-<wire x1="7.62" y1="27.94" x2="7.62" y2="30.48" width="0.1524" layer="91"/>
 <pinref part="C3" gate="G$1" pin="2"/>
+<wire x1="7.62" y1="30.48" x2="7.62" y2="27.94" width="0.1524" layer="91"/>
 </segment>
 <segment>
@@
 <segment>
 <pinref part="GND38" gate="1" pin="GND"/>
-<wire x1="226.06" y1="-10.16" x2="241.3" y2="-10.16" width="0.1524" layer="91"/>
+<wire x1="223.52" y1="-12.7" x2="231.14" y2="-12.7" width="0.1524" layer="91"/>
 <pinref part="R10" gate="G$1" pin="1"/>
+<wire x1="241.3" y1="-12.7" x2="241.3" y2="-10.16" width="0.1524" layer="91"/>
+<wire x1="231.14" y1="-7.62" x2="231.14" y2="-12.7" width="0.1524" layer="91"/>
+<wire x1="231.14" y1="-12.7" x2="231.14" y2="-30.48" width="0.1524" layer="91"/>
+<wire x1="231.14" y1="-30.48" x2="261.62" y2="-30.48" width="0.1524" layer="91"/>
+<wire x1="261.62" y1="-30.48" x2="261.62" y2="-17.78" width="0.1524" layer="91"/>
+<pinref part="C10" gate="G$1" pin="2"/>
+<pinref part="U$7" gate="G$1" pin="S"/>
+<wire x1="241.3" y1="-12.7" x2="231.14" y2="-12.7" width="0.1524" layer="91"/>
 </segment>
 <segment>
@@
 <segment>
 <pinref part="GND35" gate="1" pin="GND"/>
-<wire x1="236.22" y1="104.14" x2="251.46" y2="104.14" width="0.1524" layer="91"/>
 <pinref part="R17" gate="G$1" pin="1"/>
+<wire x1="233.68" y1="101.6" x2="241.3" y2="101.6" width="0.1524" layer="91"/>
+<wire x1="251.46" y1="101.6" x2="251.46" y2="104.14" width="0.1524" layer="91"/>
+<wire x1="241.3" y1="101.6" x2="241.3" y2="83.82" width="0.1524" layer="91"/>
+<wire x1="241.3" y1="83.82" x2="271.78" y2="83.82" width="0.1524" layer="91"/>
+<wire x1="271.78" y1="83.82" x2="271.78" y2="96.52" width="0.1524" layer="91"/>
+<pinref part="C24" gate="G$1" pin="2"/>
+<pinref part="U$16" gate="G$1" pin="S"/>
+<wire x1="251.46" y1="101.6" x2="241.3" y2="101.6" width="0.1524" layer="91"/>
+<wire x1="241.3" y1="101.6" x2="241.3" y2="106.68" width="0.1524" layer="91"/>
 </segment>
 <segment>
@@
 <segment>
 <pinref part="GND37" gate="1" pin="GND"/>
-<wire x1="-99.06" y1="101.6" x2="-83.82" y2="101.6" width="0.1524" layer="91"/>
+<wire x1="-101.6" y1="99.06" x2="-93.98" y2="99.06" width="0.1524" layer="91"/>
 <pinref part="R21" gate="G$1" pin="1"/>
+<wire x1="-93.98" y1="104.14" x2="-93.98" y2="99.06" width="0.1524" layer="91"/>
+<wire x1="-93.98" y1="99.06" x2="-93.98" y2="81.28" width="0.1524" layer="91"/>
+<wire x1="-93.98" y1="81.28" x2="-63.5" y2="81.28" width="0.1524" layer="91"/>
+<wire x1="-63.5" y1="81.28" x2="-63.5" y2="93.98" width="0.1524" layer="91"/>
+<pinref part="C30" gate="G$1" pin="2"/>
+<pinref part="U$18" gate="G$1" pin="S"/>
+<wire x1="-83.82" y1="99.06" x2="-93.98" y2="99.06" width="0.1524" layer="91"/>
 </segment>
 <segment>
@@
 <segment>
 <pinref part="GND46" gate="1" pin="GND"/>
-<wire x1="-101.6" y1="-43.18" x2="-86.36" y2="-43.18" width="0.1524" layer="91"/>
+<wire x1="-104.14" y1="-45.72" x2="-96.52" y2="-45.72" width="0.1524" layer="91"/>
 <pinref part="R23" gate="G$1" pin="1"/>
+<wire x1="-86.36" y1="-45.72" x2="-86.36" y2="-43.18" width="0.1524" layer="91"/>
+<wire x1="-96.52" y1="-40.64" x2="-96.52" y2="-45.72" width="0.1524" layer="91"/>
+<wire x1="-96.52" y1="-45.72" x2="-96.52" y2="-63.5" width="0.1524" layer="91"/>
+<wire x1="-96.52" y1="-63.5" x2="-66.04" y2="-63.5" width="0.1524" layer="91"/>
+<wire x1="-66.04" y1="-63.5" x2="-66.04" y2="-50.8" width="0.1524" layer="91"/>
+<pinref part="C34" gate="G$1" pin="2"/>
+<pinref part="U$20" gate="G$1" pin="S"/>
+<wire x1="-86.36" y1="-45.72" x2="-96.52" y2="-45.72" width="0.1524" layer="91"/>
 </segment>
 <segment>
@@
 <wire x1="-78.74" y1="124.46" x2="-104.14" y2="124.46" width="0.1524" layer="91"/>
 <wire x1="-78.74" y1="124.46" x2="-78.74" y2="114.3" width="0.1524" layer="91"/>
-<wire x1="-83.82" y1="111.76" x2="-78.74" y2="111.76" width="0.1524" layer="91"/>
+<wire x1="-83.82" y1="109.22" x2="-78.74" y2="111.76" width="0.1524" layer="91"/>
 <wire x1="-78.74" y1="111.76" x2="-78.74" y2="91.44" width="0.1524" layer="91"/>
 <wire x1="-78.74" y1="91.44" x2="-73.66" y2="91.44" width="0.1524" layer="91"/>
@@
 </segment>
 </net>
-<net name="N$16" class="0">
-<segment>
-<wire x1="231.14" y1="-7.62" x2="231.14" y2="-30.48" width="0.1524" layer="91"/>
-<wire x1="231.14" y1="-30.48" x2="261.62" y2="-30.48" width="0.1524" layer="91"/>
-<wire x1="261.62" y1="-30.48" x2="261.62" y2="-17.78" width="0.1524" layer="91"/>
-<pinref part="C10" gate="G$1" pin="2"/>
-<pinref part="U$7" gate="G$1" pin="S"/>
-</segment>
-</net>
 <net name="N$17" class="0">
 <segment>
@@
 </segment>
 </net>
-<net name="N$15" class="0">
-<segment>
-<wire x1="241.3" y1="106.68" x2="241.3" y2="83.82" width="0.1524" layer="91"/>
-<wire x1="241.3" y1="83.82" x2="271.78" y2="83.82" width="0.1524" layer="91"/>
-<wire x1="271.78" y1="83.82" x2="271.78" y2="96.52" width="0.1524" layer="91"/>
-<pinref part="C24" gate="G$1" pin="2"/>
-<pinref part="U$16" gate="G$1" pin="S"/>
-</segment>
-</net>
-<net name="N$18" class="0">
-<segment>
-<wire x1="-93.98" y1="104.14" x2="-93.98" y2="81.28" width="0.1524" layer="91"/>
-<wire x1="-93.98" y1="81.28" x2="-63.5" y2="81.28" width="0.1524" layer="91"/>
-<wire x1="-63.5" y1="81.28" x2="-63.5" y2="93.98" width="0.1524" layer="91"/>
-<pinref part="C30" gate="G$1" pin="2"/>
-<pinref part="U$18" gate="G$1" pin="S"/>
-</segment>
-</net>
-<net name="N$28" class="0">
-<segment>
-<wire x1="-96.52" y1="-40.64" x2="-96.52" y2="-63.5" width="0.1524" layer="91"/>
-<wire x1="-96.52" y1="-63.5" x2="-66.04" y2="-63.5" width="0.1524" layer="91"/>
-<wire x1="-66.04" y1="-63.5" x2="-66.04" y2="-50.8" width="0.1524" layer="91"/>
-<pinref part="C34" gate="G$1" pin="2"/>
-<pinref part="U$20" gate="G$1" pin="S"/>
-</segment>
-</net>
