File: quadcopter.sch (EAGLE design)
At the start: 65 parts, among them J1 ISP, U2 ATMEGA128RFA1

Commit message: autorouting works, things are good
Connections:
- net BAT_GND: now also C13.2, C28.2, STEP_DOWN.GND
- net GND: no longer C13.2, C28.2, STEP_DOWN.GND
Changed lines of the file:
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@@
 <part name="GND42" library="quadparts_prebuilt" deviceset="BAT_GND" device=""/>
 <part name="GND27" library="quadparts_prebuilt" deviceset="GND" device=""/>
-<part name="GND41" library="quadparts_prebuilt" deviceset="GND" device=""/>
 <part name="GND16" library="quadparts_prebuilt" deviceset="GND" device=""/>
 <part name="GND17" library="quadparts_prebuilt" deviceset="GND" device=""/>
@@
 <part name="B2" library="quadparts_prebuilt" deviceset="BALUN" device="0805"/>
 <part name="C13" library="quadparts_prebuilt" deviceset="CAPACITOR-NP_" device="SMD-2012-0805_CERAMIC-0.01UF" value="0.01uF"/>
-<part name="GND20" library="quadparts_prebuilt" deviceset="GND" device=""/>
 <part name="U$3" library="quadparts_prebuilt" deviceset="ANTENNA2" device="SMD5"/>
 <part name="Y2" library="quadparts_prebuilt" deviceset="CRYSTAL" device="5X3"/>
@@
 <instance part="GND42" gate="1" x="91.44" y="147.32"/>
 <instance part="GND27" gate="1" x="-10.16" y="134.62"/>
-<instance part="GND41" gate="1" x="58.42" y="144.78"/>
 <instance part="GND16" gate="1" x="116.84" y="-73.66"/>
 <instance part="GND17" gate="1" x="114.3" y="-27.94"/>
@@
 <instance part="B2" gate="G$1" x="91.44" y="0" rot="MR0"/>
 <instance part="C13" gate="G$1" x="53.34" y="137.16"/>
-<instance part="GND20" gate="1" x="53.34" y="127"/>
 <instance part="U$3" gate="G$1" x="109.22" y="12.7"/>
 <instance part="Y2" gate="G$1" x="60.96" y="-30.48"/>
@@
 </segment>
 <segment>
-<pinref part="C28" gate="G$1" pin="2"/>
-<pinref part="GND41" gate="1" pin="GND"/>
-</segment>
-<segment>
 <pinref part="C11" gate="G$1" pin="2"/>
 <pinref part="GND16" gate="1" pin="GND"/>
@@
 </segment>
 <segment>
-<pinref part="GND20" gate="1" pin="GND"/>
-<pinref part="C13" gate="G$1" pin="2"/>
-<wire x1="53.34" y1="129.54" x2="53.34" y2="132.08" width="0.1524" layer="91"/>
-</segment>
-<segment>
-<pinref part="STEP_DOWN" gate="G$1" pin="GND"/>
-<wire x1="30.48" y1="149.86" x2="20.32" y2="149.86" width="0.1524" layer="91"/>
-<label x="20.32" y="149.86" size="1.778" layer="95"/>
-</segment>
-<segment>
 <wire x1="38.1" y1="-33.02" x2="48.26" y2="-33.02" width="0.1524" layer="91"/>
 <label x="50.8" y="-33.02" size="1.27" layer="95" rot="MR180" xref="yes"/>
@@
 <wire x1="7.62" y1="139.7" x2="7.62" y2="147.32" width="0.1524" layer="91"/>
 <pinref part="GND25" gate="1" pin="BAT_GND"/>
-</segment>
-<segment>
+<pinref part="STEP_DOWN" gate="G$1" pin="GND"/>
+<wire x1="30.48" y1="149.86" x2="12.7" y2="149.86" width="0.1524" layer="91"/>
+<wire x1="12.7" y1="149.86" x2="12.7" y2="147.32" width="0.1524" layer="91"/>
+<wire x1="12.7" y1="147.32" x2="10.16" y2="147.32" width="0.1524" layer="91"/>
+<pinref part="C13" gate="G$1" pin="2"/>
+<wire x1="10.16" y1="147.32" x2="7.62" y2="147.32" width="0.1524" layer="91"/>
+<wire x1="53.34" y1="129.54" x2="53.34" y2="132.08" width="0.1524" layer="91"/>
+<wire x1="53.34" y1="129.54" x2="10.16" y2="129.54" width="0.1524" layer="91"/>
+<wire x1="10.16" y1="129.54" x2="10.16" y2="147.32" width="0.1524" layer="91"/>
+<pinref part="C28" gate="G$1" pin="2"/>
+<wire x1="58.42" y1="147.32" x2="55.88" y2="147.32" width="0.1524" layer="91"/>
+<wire x1="55.88" y1="147.32" x2="55.88" y2="129.54" width="0.1524" layer="91"/>
+<wire x1="55.88" y1="129.54" x2="53.34" y2="129.54" width="0.1524" layer="91"/>
+</segment>
+<segment>

Commit message: almost forgot newest board and schematic
Parts:
- added SW1: PUSHBUTTON_SMD-VERTICAL-1, quadparts_prebuilt:PUSHBUTTON_SMD-VERTICAL-1
Connections:
- net GND: now also SW1.1
- net RESET: now also SW1.2
Changed lines of the file:
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@@
 <part name="GND22" library="quadparts_prebuilt" deviceset="GND" device=""/>
 <part name="U2" library="quadparts_prebuilt" deviceset="ATMEGA128RFA1" device=""/>
+<part name="SW1" library="quadparts_prebuilt" deviceset="PUSHBUTTON_" device="SMD-VERTICAL-1"/>
+<part name="GND20" library="quadparts_prebuilt" deviceset="GND" device=""/>
 </parts>
 <sheets>
@@
 <instance part="GND22" gate="1" x="124.46" y="76.2"/>
 <instance part="U2" gate="G$1" x="10.16" y="-27.94" rot="MR0"/>
+<instance part="SW1" gate="G$1" x="30.48" y="35.56"/>
+<instance part="GND20" gate="1" x="17.78" y="30.48"/>
 </instances>
 <busses>
@@
 <pinref part="GND22" gate="1" pin="GND"/>
 </segment>
+<segment>
+<pinref part="GND20" gate="1" pin="GND"/>
+<pinref part="SW1" gate="G$1" pin="1"/>
+<wire x1="17.78" y1="33.02" x2="25.4" y2="33.02" width="0.1524" layer="91"/>
+</segment>
 </net>
 <net name="N$3" class="0">
@@
 <net name="RESET" class="0">
 <segment>
-<wire x1="38.1" y1="5.08" x2="50.8" y2="5.08" width="0.1524" layer="91"/>
+<wire x1="38.1" y1="5.08" x2="48.26" y2="5.08" width="0.1524" layer="91"/>
+<wire x1="48.26" y1="5.08" x2="50.8" y2="5.08" width="0.1524" layer="91"/>
 <wire x1="50.8" y1="5.08" x2="50.8" y2="7.62" width="0.1524" layer="91"/>
 <wire x1="50.8" y1="5.08" x2="53.34" y2="5.08" width="0.1524" layer="91"/>
@@
 <pinref part="R1" gate="G$1" pin="1"/>
 <pinref part="U2" gate="G$1" pin="RSTN"/>
+<pinref part="SW1" gate="G$1" pin="2"/>
+<wire x1="35.56" y1="33.02" x2="48.26" y2="33.02" width="0.1524" layer="91"/>
+<wire x1="48.26" y1="33.02" x2="48.26" y2="5.08" width="0.1524" layer="91"/>
 </segment>
 <segment>
@@
 <segment>
 <wire x1="177.8" y1="-68.58" x2="182.88" y2="-68.58" width="0.1524" layer="91"/>
-<label x="182.88" y="-68.58" size="1.778" layer="95" rot="R90"/>
+<label x="182.88" y="-63.5" size="1.778" layer="95" rot="R180"/>
 <pinref part="R7" gate="G$1" pin="1"/>
+<wire x1="182.88" y1="-68.58" x2="182.88" y2="-66.04" width="0.1524" layer="91"/>
 </segment>
 <segment>
 <wire x1="170.18" y1="-40.64" x2="170.18" y2="-50.8" width="0.1524" layer="91"/>
-<label x="170.18" y="-50.8" size="1.778" layer="95"/>
+<label x="172.72" y="-45.72" size="1.778" layer="95"/>
 <pinref part="U$1" gate="G$1" pin="P$5.SDO_A/G"/>
-</segment>
-<segment>
-<wire x1="187.96" y1="7.62" x2="193.04" y2="7.62" width="0.1524" layer="91"/>
-<label x="195.58" y="7.62" size="1.778" layer="95"/>
-<pinref part="U$1" gate="G$1" pin="P$13.DEN_A/G"/>
+<wire x1="170.18" y1="-50.8" x2="172.72" y2="-50.8" width="0.1524" layer="91"/>
+<wire x1="172.72" y1="-50.8" x2="172.72" y2="-48.26" width="0.1524" layer="91"/>
 </segment>
 <segment>
@@
 <junction x="187.96" y="-10.16"/>
 <pinref part="U$1" gate="G$1" pin="P$6.SDO_M"/>
-<label x="195.58" y="-10.16" size="1.778" layer="95"/>
-</segment>
-<segment>
+<wire x1="187.96" y1="7.62" x2="193.04" y2="7.62" width="0.1524" layer="91"/>
+<label x="193.04" y="12.7" size="1.778" layer="95"/>
+<pinref part="U$1" gate="G$1" pin="P$13.DEN_A/G"/>
+<wire x1="193.04" y1="7.62" x2="193.04" y2="10.16" width="0.1524" layer="91"/>
+<wire x1="193.04" y1="-10.16" x2="193.04" y2="7.62" width="0.1524" layer="91"/>
+</segment>
+<segment>
